Commit message: working tm and ur as preview only scene effects

File: uni_pal_description/urdf/pallet_right.urdf (robot description, URDF)
Before this commit: robot pallet_right, 1 links, 1 joints
Links:
- link pallet_right: geometry collision box size=0.784 0.984 1.180; visual box size=0.784 0.984 1.180

File: uni_pal_description/urdf/station.urdf (robot description, URDF)
Before this commit: robot station, 1 links, 1 joints
Links:
- link station: geometry collision box size=0.784 0.984 1.180; visual box size=0.784 0.984 1.180
