Commit message: working sim with ursim

File: uni_pal_description/urdf/gripper.urdf (robot description, URDF)
Before this commit: robot gripper, 1 links, 1 joints
Links:
- link gripper: geometry collision mesh filename=file://$(find uni_pal_description)/meshes/Chwytak_50065.stl scale=10 10 10; visual mesh filename=file://$(find uni_pal_description)/meshes/Chwytak_50065.stl scale=10 10 10
Joints:
- joint flange - gripper: origin xyz=0.03 0.0 0.0 rpy=0.0 0.0 3.14 -> xyz=0.1 0.0 0.0 rpy=0.0 0.0 3.14

File: uni_pal_description/urdf/pallet.urdf (robot description, URDF)
Before this commit: robot pallet_right, 1 links, 1 joints
Links:
- removed link pallet_right
- added link pallet; collision mesh filename=file://$(find uni_pal_description)/meshes/Paleta_small.stl scale=0.784 0.984 1.180; visual mesh filename=file://$(find uni_pal_description)/meshes/Paleta_small.stl scale=0.784 0.984 1.180
Joints:
- removed joint world - pallet_right
- added joint world - pallet: type fixed, parent world, child pallet, origin xyz=-1.2 -1.0 0.0 rpy=0.0 0.0 0.0

File: uni_pal_description/urdf/robot.urdf.xacro (robot description, xacro)
@@ -1,12 +1,13 @@
 <?xml version="1.0"?>
-<robot xmlns:xacro="http://wiki.ros.org/xacro" name="ur20">
-  <xacro:arg name="name" default="ur20"/>
+<robot xmlns:xacro="http://wiki.ros.org/xacro" name="ur10">
+  <xacro:arg name="name" default="ur10"/>
   <link name="world" />
-	<xacro:include filename="$(find uni_pal_description)/urdf/pallet_left.urdf"/>
-	<xacro:include filename="$(find uni_pal_description)/urdf/pallet_right.urdf"/>
+	<xacro:include filename="$(find uni_pal_description)/urdf/pallet.urdf"/>
+	<xacro:include filename="$(find uni_pal_description)/urdf/box_slipsheets.urdf"/>
+	<xacro:include filename="$(find uni_pal_description)/urdf/box_tape.urdf"/>
 	<xacro:include filename="$(find uni_pal_description)/urdf/station.urdf"/>
   <!-- import main macro -->
   <xacro:include filename="$(find ur_description)/urdf/ur_macro.xacro"/>
-  <xacro:arg name="ur_type" default="ur20"/>
+  <xacro:arg name="ur_type" default="ur10"/>
   <!-- parameters -->
   <xacro:arg name="tf_prefix" default="" />
@@ -90,9 +91,6 @@
     trajectory_port="$(arg trajectory_port)"
     >
-    <origin xyz="0.075 0.0 0.71" rpy="0.0 0.0 0.0" />          <!-- position robot in the world -->
+    <origin xyz="0.0 0.0 0.99" rpy="0.0 0.0 0.0" />          <!-- position robot in the world -->
   </xacro:ur_robot>
-	<xacro:include filename="$(find uni_pal_description)/urdf/padding_j3.urdf"/>
-	<xacro:include filename="$(find uni_pal_description)/urdf/padding_j4.urdf"/>
-	<xacro:include filename="$(find uni_pal_description)/urdf/padding_j5.urdf"/>
 	<xacro:include filename="$(find uni_pal_description)/urdf/gripper.urdf"/>
 </robot>

File: uni_pal_description/urdf/station.urdf (robot description, URDF)
Before this commit: robot station, 1 links, 1 joints
Links:
- link station: geometry collision mesh filename=file://$(find uni_pal_description)/meshes/station.stl scale=10 10 10; visual mesh filename=file://$(find uni_pal_description)/meshes/station.stl scale=10 10 10
Joints:
- joint world - station: origin xyz=0.0 0.0 0.0 rpy=0.0 0.0 -1.57 -> xyz=0.0 0.0 0.0 rpy=0.0 0.0 3.1415

Commit message: working moveit visu on both, but changes in rviz needed

File: uni_pal_description/urdf/gripper.urdf (robot description, URDF)
Before this commit: robot gripper, 1 links, 1 joints
Links:
- link gripper: geometry collision mesh filename=file://$(find uni_pal_description)/meshes/gripper.stl scale=1.0 1.0 1.0; visual mesh filename=file://$(find uni_pal_description)/meshes/gripper.stl scale=1.0 1.0 1.0
Joints:
- joint flange - gripper: origin xyz=0.1 0.0 0.0 rpy=0.0 0.0 3.14 -> xyz=0.03 0.0 0.0 rpy=0.0 0.0 3.14

File: uni_pal_description/urdf/pallet_right.urdf (robot description, URDF)
Before this commit: robot pallet, 1 links, 1 joints
Links:
- removed link pallet
- added link pallet_right; collision mesh filename=file://$(find uni_pal_description)/meshes/Paleta_small.stl scale=0.784 0.984 1.180; visual mesh filename=file://$(find uni_pal_description)/meshes/Paleta_small.stl scale=0.784 0.984 1.180
Joints:
- removed joint world - pallet
- added joint world - pallet_right: type fixed, parent world, child pallet_right, origin xyz=0.289 -0.65 0.0 rpy=0.0 0.0 0.0

File: uni_pal_description/urdf/robot.urdf.xacro (robot description, xacro)
@@ -1,13 +1,12 @@
 <?xml version="1.0"?>
-<robot xmlns:xacro="http://wiki.ros.org/xacro" name="ur20">
-  <xacro:arg name="name" default="ur20"/>
+<robot xmlns:xacro="http://wiki.ros.org/xacro" name="ur10">
+  <xacro:arg name="name" default="ur10"/>
   <link name="world" />
-	<xacro:include filename="$(find uni_pal_description)/urdf/pallet.urdf"/>
-	<xacro:include filename="$(find uni_pal_description)/urdf/box_slipsheets.urdf"/>
-	<xacro:include filename="$(find uni_pal_description)/urdf/box_tape.urdf"/>
+	<xacro:include filename="$(find uni_pal_description)/urdf/pallet_left.urdf"/>
+	<xacro:include filename="$(find uni_pal_description)/urdf/pallet_right.urdf"/>
 	<xacro:include filename="$(find uni_pal_description)/urdf/station.urdf"/>
   <!-- import main macro -->
   <xacro:include filename="$(find ur_description)/urdf/ur_macro.xacro"/>
-  <xacro:arg name="ur_type" default="ur20"/>
+  <xacro:arg name="ur_type" default="ur10"/>
   <!-- parameters -->
   <xacro:arg name="tf_prefix" default="" />
@@ -91,6 +90,9 @@
     trajectory_port="$(arg trajectory_port)"
     >
-    <origin xyz="0.0 0.0 0.99" rpy="0.0 0.0 0.0" />          <!-- position robot in the world -->
+    <origin xyz="0.075 0.0 0.71" rpy="0.0 0.0 0.0" />          <!-- position robot in the world -->
   </xacro:ur_robot>
+	<xacro:include filename="$(find uni_pal_description)/urdf/padding_j3.urdf"/>
+	<xacro:include filename="$(find uni_pal_description)/urdf/padding_j4.urdf"/>
+	<xacro:include filename="$(find uni_pal_description)/urdf/padding_j5.urdf"/>
 	<xacro:include filename="$(find uni_pal_description)/urdf/gripper.urdf"/>
 </robot>

File: uni_pal_description/urdf/station.urdf (robot description, URDF)
Before this commit: robot station, 1 links, 1 joints
Links:
- link station: geometry collision mesh filename=file://$(find uni_pal_description)/meshes/base.stl scale=1.0 1.0 1.0; visual mesh filename=file://$(find uni_pal_description)/meshes/base.stl scale=1.0 1.0 1.0
Joints:
- joint world - station: origin xyz=0.0 0.0 0.0 rpy=0.0 0.0 3.1415 -> xyz=0.0 0.0 0.0 rpy=0.0 0.0 -1.57
