Commit message: added readme about config.yaml & mesh copy file working

File: uni_pal_description/urdf/pallet_left.urdf (robot description, URDF)
Before this commit: robot pallet_left, 1 links, 1 joints
Links:
- link pallet_left: geometry collision mesh filename=file://$(find uni_pal_description)/meshes/Paleta_small.stl; visual mesh filename=file://$(find uni_pal_description)/meshes/Paleta_small.stl

File: uni_pal_description/urdf/robot.urdf.xacro (robot description, xacro)
@@ -5,91 +5,92 @@
 	<xacro:include filename="$(find uni_pal_description)/urdf/pallet_left.urdf"/>
 	<xacro:include filename="$(find uni_pal_description)/urdf/pallet_right.urdf"/>
+	<xacro:include filename="$(find uni_pal_description)/urdf/station.urdf"/>
    <!-- import main macro -->
-   <xacro:include filename="$(find ur_description)/urdf/ur_macro.xacro"/>
-   <!-- possible 'ur_type' values: ur3, ur3e, ur5, ur5e, ur10, ur10e, ur16e, ur20, ur30 -->
-   <!-- the default value should raise an error in case this was called without defining the type -->
-   <xacro:arg name="ur_type" default="ur5x"/>
-   <!-- parameters -->
-   <xacro:arg name="tf_prefix" default="" />
-   <xacro:arg name="joint_limit_params" default="$(find ur_description)/config/$(arg ur_type)/joint_limits.yaml"/>
-   <xacro:arg name="kinematics_params" default="$(find ur_description)/config/$(arg ur_type)/default_kinematics.yaml"/>
-   <xacro:arg name="physical_params" default="$(find ur_description)/config/$(arg ur_type)/physical_parameters.yaml"/>
-   <xacro:arg name="visual_params" default="$(find ur_description)/config/$(arg ur_type)/visual_parameters.yaml"/>
-   <xacro:arg name="transmission_hw_interface" default=""/>
-   <xacro:arg name="safety_limits" default="false"/>
-   <xacro:arg name="safety_pos_margin" default="0.15"/>
-   <xacro:arg name="safety_k_position" default="20"/>
-   <!-- ros2_control related parameters -->
-   <xacro:arg name="headless_mode" default="false" />
-   <xacro:arg name="robot_ip" default="0.0.0.0" />
-   <xacro:arg name="script_filename" default=""/>
-   <xacro:arg name="output_recipe_filename" default=""/>
-   <xacro:arg name="input_recipe_filename" default=""/>
-   <xacro:arg name="reverse_ip" default="0.0.0.0"/>
-   <xacro:arg name="script_command_port" default="50004"/>
-   <xacro:arg name="reverse_port" default="50001"/>
-   <xacro:arg name="script_sender_port" default="50002"/>
-   <xacro:arg name="trajectory_port" default="50003"/>
-   <!--   tool communication related parameters-->
-   <xacro:arg name="use_tool_communication" default="false" />
-   <xacro:arg name="tool_voltage" default="0" />
-   <xacro:arg name="tool_parity" default="0" />
-   <xacro:arg name="tool_baud_rate" default="115200" />
-   <xacro:arg name="tool_stop_bits" default="1" />
-   <xacro:arg name="tool_rx_idle_chars" default="1.5" />
-   <xacro:arg name="tool_tx_idle_chars" default="3.5" />
-   <xacro:arg name="tool_device_name" default="/tmp/ttyUR" />
-   <xacro:arg name="tool_tcp_port" default="54321" />
-     <!-- Simulation parameters -->
-   <xacro:arg name="use_fake_hardware" default="false" />
-   <xacro:arg name="fake_sensor_commands" default="false" />
-   <xacro:arg name="sim_gazebo" default="false" />
-   <xacro:arg name="sim_ignition" default="false" />
-   <xacro:arg name="simulation_controllers" default="" />
-   <!-- initial position for simulations (Fake Hardware, Gazebo, Ignition) -->
-   <xacro:arg name="initial_positions_file" default="$(find ur_description)/config/initial_positions.yaml"/>
-   <!-- convert to property to use substitution in function -->
-   <xacro:property name="initial_positions_file" default="$(arg initial_positions_file)"/>
-   <xacro:property name="is_sim_gazebo" value="$(arg sim_gazebo)"/>
-   <xacro:property name="is_sim_ignition" value="$(arg sim_ignition)"/>
-   <!-- arm -->
-   <xacro:ur_robot
-     name="$(arg name)"
-     tf_prefix="$(arg tf_prefix)"
-     parent="world"
-     joint_limits_parameters_file="$(arg joint_limit_params)"
-     kinematics_parameters_file="$(arg kinematics_params)"
-     physical_parameters_file="$(arg physical_params)"
-     visual_parameters_file="$(arg visual_params)"
-     transmission_hw_interface="$(arg transmission_hw_interface)"
-     safety_limits="$(arg safety_limits)"
-     safety_pos_margin="$(arg safety_pos_margin)"
-     safety_k_position="$(arg safety_k_position)"
-     use_fake_hardware="$(arg use_fake_hardware)"
-     fake_sensor_commands="$(arg fake_sensor_commands)"
-     sim_gazebo="$(arg sim_gazebo)"
-     sim_ignition="$(arg sim_ignition)"
-     headless_mode="$(arg headless_mode)"
-     initial_positions="${xacro.load_yaml(initial_positions_file)}"
-     use_tool_communication="$(arg use_tool_communication)"
-     tool_voltage="$(arg tool_voltage)"
-     tool_parity="$(arg tool_parity)"
-     tool_baud_rate="$(arg tool_baud_rate)"
-     tool_stop_bits="$(arg tool_stop_bits)"
-     tool_rx_idle_chars="$(arg tool_rx_idle_chars)"
-     tool_tx_idle_chars="$(arg tool_tx_idle_chars)"
-     tool_device_name="$(arg tool_device_name)"
-     tool_tcp_port="$(arg tool_tcp_port)"
-     robot_ip="$(arg robot_ip)"
-     script_filename="$(arg script_filename)"
-     output_recipe_filename="$(arg output_recipe_filename)"
-     input_recipe_filename="$(arg input_recipe_filename)"
-     reverse_ip="$(arg reverse_ip)"
-     script_command_port="$(arg script_command_port)"
-     reverse_port="$(arg reverse_port)"
-     script_sender_port="$(arg script_sender_port)"
-     trajectory_port="$(arg trajectory_port)"
-     >
-     <origin xyz="0 0 0" rpy="0 0 0" />          <!-- position robot in the world -->
-   </xacro:ur_robot>
+      <xacro:include filename="$(find ur_description)/urdf/ur_macro.xacro"/>
+      <!-- possible 'ur_type' values: ur3, ur3e, ur5, ur5e, ur10, ur10e, ur16e, ur20, ur30 -->
+      <!-- the default value should raise an error in case this was called without defining the type -->
+      <xacro:arg name="ur_type" default="ur5x"/>
+      <!-- parameters -->
+      <xacro:arg name="tf_prefix" default="" />
+      <xacro:arg name="joint_limit_params" default="$(find ur_description)/config/$(arg ur_type)/joint_limits.yaml"/>
+      <xacro:arg name="kinematics_params" default="$(find ur_description)/config/$(arg ur_type)/default_kinematics.yaml"/>
+      <xacro:arg name="physical_params" default="$(find ur_description)/config/$(arg ur_type)/physical_parameters.yaml"/>
+      <xacro:arg name="visual_params" default="$(find ur_description)/config/$(arg ur_type)/visual_parameters.yaml"/>
+      <xacro:arg name="transmission_hw_interface" default=""/>
+      <xacro:arg name="safety_limits" default="false"/>
+      <xacro:arg name="safety_pos_margin" default="0.15"/>
+      <xacro:arg name="safety_k_position" default="20"/>
+      <!-- ros2_control related parameters -->
+      <xacro:arg name="headless_mode" default="false" />
+      <xacro:arg name="robot_ip" default="0.0.0.0" />
+      <xacro:arg name="script_filename" default=""/>
+      <xacro:arg name="output_recipe_filename" default=""/>
+      <xacro:arg name="input_recipe_filename" default=""/>
+      <xacro:arg name="reverse_ip" default="0.0.0.0"/>
+      <xacro:arg name="script_command_port" default="50004"/>
+      <xacro:arg name="reverse_port" default="50001"/>
+      <xacro:arg name="script_sender_port" default="50002"/>
+      <xacro:arg name="trajectory_port" default="50003"/>
+      <!--   tool communication related parameters-->
+      <xacro:arg name="use_tool_communication" default="false" />
+      <xacro:arg name="tool_voltage" default="0" />
+      <xacro:arg name="tool_parity" default="0" />
+      <xacro:arg name="tool_baud_rate" default="115200" />
+      <xacro:arg name="tool_stop_bits" default="1" />
+      <xacro:arg name="tool_rx_idle_chars" default="1.5" />
+      <xacro:arg name="tool_tx_idle_chars" default="3.5" />
+      <xacro:arg name="tool_device_name" default="/tmp/ttyUR" />
+      <xacro:arg name="tool_tcp_port" default="54321" />
+        <!-- Simulation parameters -->
+      <xacro:arg name="use_fake_hardware" default="false" />
+      <xacro:arg name="fake_sensor_commands" default="false" />
+      <xacro:arg name="sim_gazebo" default="false" />
+      <xacro:arg name="sim_ignition" default="false" />
+      <xacro:arg name="simulation_controllers" default="" />
+      <!-- initial position for simulations (Fake Hardware, Gazebo, Ignition) -->
+      <xacro:arg name="initial_positions_file" default="$(find ur_description)/config/initial_positions.yaml"/>
+      <!-- convert to property to use substitution in function -->
+      <xacro:property name="initial_positions_file" default="$(arg initial_positions_file)"/>
+      <xacro:property name="is_sim_gazebo" value="$(arg sim_gazebo)"/>
+      <xacro:property name="is_sim_ignition" value="$(arg sim_ignition)"/>
+      <!-- arm -->
+      <xacro:ur_robot
+        name="$(arg name)"
+        tf_prefix="$(arg tf_prefix)"
+        parent="world"
+        joint_limits_parameters_file="$(arg joint_limit_params)"
+        kinematics_parameters_file="$(arg kinematics_params)"
+        physical_parameters_file="$(arg physical_params)"
+        visual_parameters_file="$(arg visual_params)"
+        transmission_hw_interface="$(arg transmission_hw_interface)"
+        safety_limits="$(arg safety_limits)"
+        safety_pos_margin="$(arg safety_pos_margin)"
+        safety_k_position="$(arg safety_k_position)"
+        use_fake_hardware="$(arg use_fake_hardware)"
+        fake_sensor_commands="$(arg fake_sensor_commands)"
+        sim_gazebo="$(arg sim_gazebo)"
+        sim_ignition="$(arg sim_ignition)"
+        headless_mode="$(arg headless_mode)"
+        initial_positions="${xacro.load_yaml(initial_positions_file)}"
+        use_tool_communication="$(arg use_tool_communication)"
+        tool_voltage="$(arg tool_voltage)"
+        tool_parity="$(arg tool_parity)"
+        tool_baud_rate="$(arg tool_baud_rate)"
+        tool_stop_bits="$(arg tool_stop_bits)"
+        tool_rx_idle_chars="$(arg tool_rx_idle_chars)"
+        tool_tx_idle_chars="$(arg tool_tx_idle_chars)"
+        tool_device_name="$(arg tool_device_name)"
+        tool_tcp_port="$(arg tool_tcp_port)"
+        robot_ip="$(arg robot_ip)"
+        script_filename="$(arg script_filename)"
+        output_recipe_filename="$(arg output_recipe_filename)"
+        input_recipe_filename="$(arg input_recipe_filename)"
+        reverse_ip="$(arg reverse_ip)"
+        script_command_port="$(arg script_command_port)"
+        reverse_port="$(arg reverse_port)"
+        script_sender_port="$(arg script_sender_port)"
+        trajectory_port="$(arg trajectory_port)"
+        >
+        <origin xyz="0 0 0" rpy="0 0 0" />          <!-- position robot in the world -->
+      </xacro:ur_robot>
 </robot>

File: uni_pal_description/urdf/station.urdf (robot description, URDF)
Before this commit: robot pallet_right, 1 links, 1 joints
Links:
- removed link pallet_right
- added link station; collision box size=0.5 0.5 1.2; visual box size=0.5 0.5 1.2
Joints:
- removed joint world - pallet_right
- added joint pallet_left - station: type fixed, parent pallet_left, child station, origin xyz=0.0 0.0 0.0 rpy=0.0 0.0 0.0

Commit message: station generating, now adding robot specific cads

File: uni_pal_description/urdf/pallet_left.urdf (robot description, URDF)
Before this commit: robot pallet_left, 1 links, 1 joints
Links:
- link pallet_left: geometry collision mesh filename=file://$(find uni_pal_description)/meshes/Paleta_small.stl scale=0.784 0.984 1.180; visual mesh filename=file://$(find uni_pal_description)/meshes/Paleta_small.stl scale=0.784 0.984 1.180
Joints:
- joint world - pallet_left: origin xyz=-0.79 -0.1 0.0 rpy=0.0 0.0 0.0 -> xyz=-1.089 -0.65 0.0 rpy=0.0 0.0 0.0

File: uni_pal_description/urdf/pallet_right.urdf (robot description, URDF)
Before this commit: robot pallet_right, 1 links, 1 joints
Links:
- link pallet_right: geometry collision mesh filename=file://$(find uni_pal_description)/meshes/Paleta_small.stl scale=0.784 0.984 1.180; visual mesh filename=file://$(find uni_pal_description)/meshes/Paleta_small.stl scale=0.784 0.984 1.180
Joints:
- joint world - pallet_right: origin xyz=0.79 -0.1 0.0 rpy=0.0 0.0 0.0 -> xyz=0.289 -0.65 0.0 rpy=0.0 0.0 0.0

File: uni_pal_description/urdf/robot.urdf.xacro (robot description, xacro)
@@ -58,5 +58,5 @@
         name="$(arg name)"
         tf_prefix="$(arg tf_prefix)"
-        parent="world"
+        parent="station"
         joint_limits_parameters_file="$(arg joint_limit_params)"
         kinematics_parameters_file="$(arg kinematics_params)"
@@ -92,5 +92,5 @@
         trajectory_port="$(arg trajectory_port)"
         >
-        <origin xyz="0 0 0" rpy="0 0 0" />          <!-- position robot in the world -->
+        <origin xyz="0.075 0.0 0.71" rpy="0.0 0.0 0.0" />          <!-- position robot in the world -->
       </xacro:ur_robot>
 </robot>

File: uni_pal_description/urdf/station.urdf (robot description, URDF)
Before this commit: robot station, 1 links, 1 joints
Links:
- link station: geometry collision mesh filename=file://$(find uni_pal_description)/meshes/base.stl scale=1.0 1.0 1.0; visual mesh filename=file://$(find uni_pal_description)/meshes/base.stl scale=1.0 1.0 1.0
Joints:
- removed joint pallet_left - station
- added joint world - station: type fixed, parent world, child station, origin xyz=0.0 0.0 0.0 rpy=0.0 0.0 -1.57

Commit message: robot config for tm and ur enabled accessories for both

File: uni_pal_description/urdf/pallet_left.urdf (robot description, URDF)
Before this commit: robot pallet_right, 1 links, 1 joints
Links:
- removed link pallet_right
- added link pallet_left; collision mesh filename=file://$(find uni_pal_description)/meshes/Paleta_small.stl scale=0.784 0.984 1.180; visual mesh filename=file://$(find uni_pal_description)/meshes/Paleta_small.stl scale=0.784 0.984 1.180
Joints:
- removed joint world - pallet_right
- added joint world - pallet_left: type fixed, parent world, child pallet_left, origin xyz=-1.089 -0.65 0.0 rpy=0.0 0.0 0.0

File: uni_pal_description/urdf/robot.urdf.xacro (robot description, xacro)
@@ -1,11 +1,12 @@
 <?xml version="1.0"?>
-<robot xmlns:xacro="http://wiki.ros.org/xacro" name="ur10">
-  <xacro:arg name="name" default="ur10"/>
+<robot xmlns:xacro="http://wiki.ros.org/xacro" name="ur20">
+  <xacro:arg name="name" default="ur20"/>
   <link name="world" />
+	<xacro:include filename="$(find uni_pal_description)/urdf/pallet_left.urdf"/>
 	<xacro:include filename="$(find uni_pal_description)/urdf/pallet_right.urdf"/>
 	<xacro:include filename="$(find uni_pal_description)/urdf/station.urdf"/>
   <!-- import main macro -->
   <xacro:include filename="$(find ur_description)/urdf/ur_macro.xacro"/>
-  <xacro:arg name="ur_type" default="ur5x"/>
+  <xacro:arg name="ur_type" default="ur20"/>
   <!-- parameters -->
   <xacro:arg name="tf_prefix" default="" />
@@ -91,3 +92,7 @@
     <origin xyz="0.075 0.0 0.71" rpy="0.0 0.0 0.0" />          <!-- position robot in the world -->
   </xacro:ur_robot>
+	<xacro:include filename="$(find uni_pal_description)/urdf/padding_j3.urdf"/>
+	<xacro:include filename="$(find uni_pal_description)/urdf/padding_j4.urdf"/>
+	<xacro:include filename="$(find uni_pal_description)/urdf/padding_j5.urdf"/>
+	<xacro:include filename="$(find uni_pal_description)/urdf/gripper.urdf"/>
 </robot>

File: uni_pal_description/urdf/station.urdf (robot description, URDF)
Before this commit: robot station, 1 links, 1 joints
Links:
- link station: geometry collision mesh filename=file://$(find uni_pal_description)/meshes/base.stl scale=1.0 1.0 1.0; visual mesh filename=file://$(find uni_pal_description)/meshes/base.stl scale=1.0 1.0 1.0

Commit message: final commit before thesis defence

File: uni_pal_description/urdf/pallet_left.urdf (robot description, URDF)
Before this commit: robot pallet_left, 1 links, 1 joints
Links:
- link pallet_left: geometry collision box size=0.8 1.2 0.144; visual box size=0.8 1.2 0.144
Joints:
- joint world - pallet_left: origin xyz=-1.089 -0.65 0.0 rpy=0.0 0.0 0.0 -> xyz=-1.19 -0.7 0.0 rpy=0.0 0.0 0.0

File: uni_pal_description/urdf/pallet_right.urdf (robot description, URDF)
Before this commit: robot pallet_right, 1 links, 1 joints
Links:
- link pallet_right: geometry collision box size=1.02 1.22 0.122; visual box size=1.02 1.22 0.122
Joints:
- joint world - pallet_right: origin xyz=0.289 -0.65 0.0 rpy=0.0 0.0 0.0 -> xyz=0.39 -0.71 0.0 rpy=0.0 0.0 0.0

File: uni_pal_description/urdf/robot.urdf.xacro (robot description, xacro)
@@ -21,5 +21,5 @@
   <!-- ros2_control related parameters -->
   <xacro:arg name="headless_mode" default="false" />
-  <xacro:arg name="robot_ip" default="192.168.56.100" />
+  <xacro:arg name="robot_ip" default="192.168.56.101" />
   <xacro:arg name="script_filename" default="$(find ur_client_library)/resources/external_control.urscript"/>
   <xacro:arg name="output_recipe_filename" default="$(find ur_robot_driver)/resources/rtde_output_recipe.txt"/>
@@ -92,7 +92,3 @@
     <origin xyz="0.075 0.0 0.71" rpy="0.0 0.0 1.57" />          <!-- position robot in the world -->
   </xacro:ur_robot>
-	<xacro:include filename="$(find uni_pal_description)/urdf/padding_j3.urdf"/>
-	<xacro:include filename="$(find uni_pal_description)/urdf/padding_j4.urdf"/>
-	<xacro:include filename="$(find uni_pal_description)/urdf/padding_j5.urdf"/>
-	<xacro:include filename="$(find uni_pal_description)/urdf/gripper.urdf"/>
 </robot>
